File: PCB/ErgoKey_L/ErgoKey_L.kicad_pcb (KiCad board)
At the start: 2 copper layers, 181 x 114.3 mm, 68 parts, among them SW1 RotaryEncoder_Switch, U1 ProMicro

Commit message: worked on the right-hand side and changed dev board to nice!nano
Parts:
- removed U1: ProMicro, PCM_marbastlib-xp-promicroish:ProMicro_USBup
- added U2: nice_nano, PCM_marbastlib-xp-promicroish:nice_nano_AH_USBup, F.Cu at (192.4, 33.3)
- S1, S2, S3, S4: value MX_stab 1 x 2 -> MX_stab
- moved D10 19.1 mm to (85.7, 57.7)
- moved D13 19.1 mm to (142.9, 52.4)
- moved D17 19.1 mm to (85.7, 76.2)
- moved D20 19.1 mm to (142.9, 71.4)
- moved D23 19.1 mm to (85.7, 95.2)
- moved D26 19.1 mm to (142.9, 90.5)
- moved D29 19.1 mm to (85.7, 114.3)
- moved D3 19.1 mm to (85.7, 38.1)
- moved D6 19.1 mm to (142.9, 33.3)
- moved D16 19.1 mm to (57.1, 76.2)
- moved D22 19.1 mm to (57.1, 95.2)
- moved D9 19.1 mm to (57.1, 57.1)
- moved D15 19.1 mm to (28.6, 76.2)
- moved D8 19.1 mm to (28.6, 57.1)
- moved D1 19.0 mm to (47.6, 38.1)
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