File: PCB/ErgoKey_R/ErgoKey_R.kicad_sch (KiCad schematic)
At the start: 68 parts, among them SW1 RotaryEncoder_Switch, U2 nice_nano

Commit message: worked on the right-hand side and changed dev board to nice!nano
Parts:
- removed S4: MX_stab, PCM_marbastlib-mx:STAB_MX_2u, symbol PCM_marbastlib-mx:MX_stab
- removed SW1: RotaryEncoder_Switch, Rotary_Encoder:RotaryEncoder_Alps_EC11E-Switch_Vertical_H20mm, symbol Device:RotaryEncoder_Switch
- removed U2: nice_nano, PCM_marbastlib-xp-promicroish:nice_nano_AH_USBup, symbol PCM_marbastlib-promicroish:nice_nano
- added D32, D33: 1N4148W, Diode_SMD:D_SOD-123, symbol Diode:1N4148W
- added MX32, MX33: MX_SW_HS, PCM_marbastlib-mx:SW_MX_HS_CPG151101S11_1u, symbol PCM_marbastlib-mx:MX_SW_HS_CPG151101S11
- added U1: nice_nano, PCM_marbastlib-xp-promicroish:nice_nano_AH_USBup, symbol PCM_marbastlib-promicroish:nice_nano
Connections:
- net GND: now also U1.14 (GND)
- net RESET: now also U1.15 (RST)
- net VCC: now also U1.16 (3V3)
- net R_Row 3: now reaches D28.1 (K)
- net R_Row 3: now also D25.1 (K), D26.1 (K), D27.1 (K), D29.1 (K), D30.1 (K)
- net R_Column 3: now reaches MX28.1
- net R_Column 3: now also MX12.1, MX20.1, MX4.1, MX32.1
- removed net L_Column 0: MX1.1, MX15.1, MX8.1
- removed net L_Column 1: MX16.1, MX2.1, MX22.1, MX9.1
- removed net L_Column 2: MX10.1, MX17.1, MX23.1, MX29.1, MX3.1
- removed net L_Column 3: MX11.1, MX18.1, MX24.1, MX30.1, MX4.1
- removed net L_Column 4: MX12.1, MX19.1, MX25.1, MX5.1
- removed net L_Column 5: MX13.1, MX20.1, MX26.1, MX31.1, MX6.1
- removed net L_Column 6: MX14.1, MX21.1, MX27.1, MX7.1
- net L_Row 0 renamed R_Row 0
- net R_Row 0: now also D8.1 (K)
- net L_Row 1 renamed R_Row 1
- net R_Row 1: now also D15.1 (K), D16.1 (K); no longer D8.1 (K)
- net L_Row 2 renamed R_Row 2
- net R_Row 2: now also D22.1 (K), D23.1 (K); no longer D15.1 (K), D16.1 (K)
- removed net L_Row 3: D22.1 (K), D23.1 (K), D24.1 (K), D25.1 (K), D26.1 (K), D27.1 (K)
- removed net L_Row 4: D29.1 (K), D30.1 (K), D31.1 (K)
- new net: D32.2 (A), MX32.2
- new net: D33.2 (A), MX33.2
- new net R_Column 0: MX1.1, MX17.1, MX25.1, MX9.1
- new net R_Column 1: MX10.1, MX18.1, MX2.1, MX26.1, MX31.1
- new net R_Column 2: MX11.1, MX19.1, MX27.1, MX3.1
- new net R_Column 4: MX13.1, MX21.1, MX29.1, MX33.1, MX5.1
- new net R_Column 5: MX14.1, MX22.1, MX30.1, MX6.1
- new net R_Column 6: MX15.1, MX23.1, MX7.1
- new net R_Column 7: MX16.1, MX8.1
- new net R_Row 4: D31.1 (K), D32.1 (K), D33.1 (K)
